File: hardware/nfc_fpc/nfc_antenna_fpc.kicad_pcb (KiCad board)
At the start: 2 copper layers, 62 x 44 mm, 2 parts

Commit message: v2.1
Parts:
- U_KEY: value NTAG213_FPC -> NTAG216_FPC
Other:
- board text added: "IC: U_KEY (NTAG216) | 100% PASSIVE (0% BATTERY OPERATION)"
- board text removed: "IC: U_KEY (NTAG213/215) | 100% PASSIVE (0% BATTERY OPERATION)"
Changed lines of the file:
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@@
 	(footprint "Package_DFN_QFN:DFN-2_1.2x0.8mm_P0.65mm" (layer "B.Cu") (at 41.0 29.0 0)
 		(property "Reference" "U_KEY" (at 0 -1.5 0) (layer "B.SilkS") (effects (font (size 0.8 0.8) (thickness 0.15))))
-		(property "Value" "NTAG213_FPC" (at 0 1.5 0) (layer "B.Fab") (effects (font (size 0.7 0.7) (thickness 0.12))))
+		(property "Value" "NTAG216_FPC" (at 0 1.5 0) (layer "B.Fab") (effects (font (size 0.7 0.7) (thickness 0.12))))
 		(pad "1" smd rect (at -0.45 0.0) (size 0.40 0.60) (layers "B.Cu" "B.Mask" "B.Paste") (net 2 "NFC_KEY_COIL"))
 		(pad "2" smd rect (at  0.45 0.0) (size 0.40 0.60) (layers "B.Cu" "B.Mask" "B.Paste") (net 2 "NFC_KEY_COIL"))
@@
 	(gr_text "Size: 62.0x38.0mm Flush Fit for 65x40mm Battery" (at 41.000 34.500) (layer "F.SilkS") (effects (font (size 0.80 0.80) (thickness 0.15))))
 	(gr_text "BACK: INDEPENDENT PASSIVE ACCESS KEY COIL" (at 41.000 21.500) (layer "B.SilkS") (effects (font (size 0.90 0.90) (thickness 0.15))))
-	(gr_text "IC: U_KEY (NTAG213/215) | 100% PASSIVE (0% BATTERY OPERATION)" (at 41.000 24.500) (layer "B.SilkS") (effects (font (size 0.80 0.80) (thickness 0.15))))
+	(gr_text "IC: U_KEY (NTAG216) | 100% PASSIVE (0% BATTERY OPERATION)" (at 41.000 24.500) (layer "B.SilkS") (effects (font (size 0.80 0.80) (thickness 0.15))))
 	(gr_text "[ ATTACH 0.1mm FERRITE SHIELD OVER BATTERY BACK ]" (at 41.000 34.500) (layer "B.SilkS") (effects (font (size 0.80 0.80) (thickness 0.15))))
 )
