File: hardware/pcb_c6_slimbadge/epd_c6_slimbadge.kicad_pcb (KiCad board)
At the start: 4 copper layers, 96 x 62 mm, 86 parts, among them J1 Type-C_16P, J2 JST_1.25mm_2P, Q1 AO3400A, SW1 SK12D07, U1 ESP32-C6-MINI-1, U10 ST25DV04K, U2 USBLC6-2SC6, U3 CH224K, U4 SY6970, U5 ME6211C33M5G, U6 QMI8658C, U7 SHT40, U8 OPT3001, U9 PCF8563T, Y1 32.768kHz

Commit message: v2.1
Parts:
- C29, C30, LED1, U7, U8: moved to B.Cu
- moved C30 84.7 mm to (-1.20, 56.8)
- moved U8 84.3 mm to (-1.20, 52.6)
- moved LED1 79.1 mm to (-1.20, 22.5), turned to 180 degrees
- moved C7 33.7 mm to (5.00, 15.0)
- moved C14 14.6 mm to (3.00, 46.6)
- moved C13 11.5 mm to (3.00, 47.9)
- moved C29 9.45 mm to (-1.20, 50.8)
- moved U7 8.84 mm to (-1.20, 55.2), turned to 180 degrees
- moved C12 8.40 mm to (3.00, 49.2)
- moved C11 5.30 mm to (3.00, 50.5)
- moved C8 4.00 mm to (3.00, 54.4)
- moved C6 2.80 mm to (3.00, 44.0)
- moved C10 2.20 mm to (3.00, 51.8)
- moved C9 0.90 mm to (3.00, 53.1)
- moved C5 0.30 mm to (3.00, 45.3)
Routing:
- net RGB_DIN: track 9.60 -> 96.0 mm, vias 0 -> 2
- net EPD_RESE: track 10.2 -> 32.0 mm
- net EPD_GDR: track 17.2 -> 37.5 mm, vias 2 -> 3
- net I2C_SDA: track 169.2 -> 150.1 mm, vias 8 -> 7
- net EPD_VDD: track 12.2 -> 25.0 mm
- net EPD_VGH: track 19.0 -> 6.60 mm
- net EPD_VGL: track 19.2 -> 7.10 mm, vias 3 -> 2
- net EPD_VPP: track 13.2 -> 24.5 mm
- net PREVGL: track 26.8 -> 37.9 mm
- net EPD_VSH1: track 14.2 -> 24.0 mm
- net I2C_SCL: track 169.2 -> 160.6 mm, vias 8 -> 10
- net GND: track 173.7 -> 181.3 mm, vias 52 -> 58
- net EPD_VSL: track 16.2 -> 23.0 mm
- net EPD_BUSY: track 101.3 -> 106.9 mm
- net EPD_RST: track 127.2 -> 131.2 mm
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Other:
- board size 96 x 62 mm -> 99 x 62 mm
- board text added: "1"
- board text added: "24"
- board text removed: "SHT40"

Commit message: v2.2
Parts:
- added C35: 0.1uF, , F.Cu at (7.40, 52.2)
- added U12: FLASH_4-128MB, , F.Cu at (4.60, 56.0)
- moved C11 3.20 mm to (3.00, 47.3)
- moved C12 3.20 mm to (3.00, 46.0)
- moved C14 3.20 mm to (3.00, 43.4)
- moved C6 3.20 mm to (3.00, 40.8)
- moved C9 3.20 mm to (3.00, 49.9)
- moved J_EPD_A 3.20 mm to (8.00, 34.8)
- moved U7 3.20 mm to (-1.20, 52.0)
- moved U8 3.20 mm to (-1.20, 49.4)
- moved LED1 3.20 mm to (-1.20, 19.3)
- moved C10 3.20 mm to (3.00, 48.6)
- moved C13 3.20 mm to (3.00, 44.7)
- moved C29 3.20 mm to (-1.20, 47.6)
- moved C30 3.20 mm to (-1.20, 53.6)
- moved C5 3.20 mm to (3.00, 42.1)
- moved C8 3.20 mm to (3.00, 51.2)
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Connections:
- U1 pad 21: (no net) -> FLASH_CS
- U8 pad 2: GND -> VCC_3V3
Routing:
- net FLASH_CS: track 0.00 -> 123.9 mm, vias 0 -> 2
- net SD_MISO: track 39.0 -> 162.0 mm, vias 2 -> 3
- net SD_SCK: track 39.9 -> 160.3 mm, vias 2 -> 3
- net SD_MOSI: track 40.0 -> 160.3 mm, vias 2 -> 3
- net VCC_3V3: track 62.0 -> 116.9 mm, vias 28 -> 30
- net EPD_SCK: track 132.7 -> 123.5 mm
- net EPD_RST: track 131.2 -> 122.4 mm
- net EPD_CS: track 149.1 -> 140.6 mm
- net EPD_DIN: track 144.5 -> 136.3 mm
- net EPD_DC: track 143.1 -> 135.2 mm
- net CHIP_EN: track 50.8 -> 45.0 mm
- net RTC_INT: track 62.8 -> 58.5 mm
- net GND: track 181.3 -> 184.5 mm, vias 58 -> 62
- net I2C_SCL: track 160.6 -> 157.4 mm
- net PREVGH: track 33.2 -> 30.0 mm
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Other:
- outline, holes or cut-outs redrawn

Commit message: v2.3
Parts:
- moved C35 1.34 mm to (8.60, 52.8)
- moved U12 1.03 mm to (5.50, 56.5)
Routing:
- net VCC_3V3: track 116.9 -> 68.8 mm
- net PREVGH: track 30.0 -> 37.8 mm
- net SD_SCK: track 160.3 -> 156.9 mm, vias 3 -> 4
- net SD_MOSI: track 160.3 -> 157.8 mm
- net FLASH_CS: track 123.9 -> 126.3 mm
- net GND: track 184.5 -> 185.4 mm
- net SD_MISO: track 162.0 -> 162.5 mm, vias 3 -> 4
