File: hardware/pcb_c6_slimbadge/epd_c6_slimbadge.kicad_sch (KiCad schematic)
At the start: 88 parts, among them J1 Type-C_16P_MidMount, J2 1.25mm_2P_Battery, Q1 AO3400A, SW1 SK12D07, U1 ESP32-C6-MINI-1-N4, U10 ST25DV04K, U2 USBLC6-2SC6, U3 CH224K, U4 SY6970, U5 ME6211C33M5G, U6 QMI8658C, U7 SHT40, U8 OPT3001, U9 PCF8563T, Y1 32.768kHz

Commit message: v2.1
Parts:
- J2: value 1.25mm_2P_Battery -> SH1.0mm_2P_Battery; footprint Connector_JST:JST_GH_SM02B-GHS-TB_1x02-1MP_P1.25mm_Horizontal -> Connector_JST:JST_SH_SM02B-SRSS-TB_1x02-1MP_P1.00mm_Horizontal; LCSC C138807 -> C160404
Changed lines of the file:
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@@
 		(exclude_from_sim no) (in_bom yes) (on_board yes) (dnp no)
 		(property "Reference" "J2" (at 300.00 121.00 0) (effects (font (size 1.27 1.27))))
-		(property "Value" "1.25mm_2P_Battery" (at 300.00 129.00 0) (effects (font (size 1.27 1.27))))
-		(property "Footprint" "Connector_JST:JST_GH_SM02B-GHS-TB_1x02-1MP_P1.25mm_Horizontal" (at 300.00 125.00 0) (hide yes) (effects (font (size 1.27 1.27))))
+		(property "Value" "SH1.0mm_2P_Battery" (at 300.00 129.00 0) (effects (font (size 1.27 1.27))))
+		(property "Footprint" "Connector_JST:JST_SH_SM02B-SRSS-TB_1x02-1MP_P1.00mm_Horizontal" (at 300.00 125.00 0) (hide yes) (effects (font (size 1.27 1.27))))
 		(property "Datasheet" "~" (at 300.00 125.00 0) (hide yes) (effects (font (size 1.27 1.27))))
-		(property "Description" "" (at 300.00 125.00 0) (hide yes) (effects (font (size 1.27 1.27))))
-		(property "LCSC" "C138807" (at 300.00 125.00 0) (hide yes) (effects (font (size 1.27 1.27))))
+		(property "Description" "JST SH 1.0mm 2P Horizontal SMD" (at 300.00 125.00 0) (hide yes) (effects (font (size 1.27 1.27))))
+		(property "LCSC" "C160404" (at 300.00 125.00 0) (hide yes) (effects (font (size 1.27 1.27))))
 		(pin "1")
 		(pin "2")

Commit message: cleanup
Parts:
- added C35: 0.1uF, Capacitor_SMD:C_0402_1005Metric, symbol Device:C
- added U12: W25Q128JVSIQ(Optional_Flash), Package_SO:SOIC-8_208mil_WSON-8_8x6mm_DualCombo, symbol Memory_Flash:W25Q128JV
Connections:
- net EP: now also C35.2, U12.4 (GND)
- net SD_MISO: now also U12.2 (DO(IO1))
- net SD_MOSI: now also U12.5 (DI(IO0))
- net SD_SCK: now also U12.6 (CLK)
- net VCC_3V3: now also C35.1, U12.3 (~{WP}(IO2)), U12.7 (~{HOLD}(IO3)), U12.8 (VCC)
- new net FLASH_CS: U12.1 (~{CS})
Changed lines of the file:
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@@
 	(label "SD_MISO" (at 122.86 100.00 0) (fields_autoplaced yes)
+		(effects (font (size 1.27 1.27)) (justify left bottom)))
+		(label "FLASH_CS" (at 122.86 102.54 0) (fields_autoplaced yes)
 		(effects (font (size 1.27 1.27)) (justify left bottom)))
 	(label "CHG_INT" (at 122.86 105.08 0) (fields_autoplaced yes)
@@
 		(instances (project "epd_c6_slimbadge" (path "/00000000-0000-0000-0000-000000000001" (reference "TP2") (unit 1))))
 	)
+	(label "FLASH_CS" (at 262.30 232.38 180) (fields_autoplaced yes)
+		(effects (font (size 1.27 1.27)) (justify left bottom)))
+	(label "SD_MISO" (at 262.30 237.46 180) (fields_autoplaced yes)
+		(effects (font (size 1.27 1.27)) (justify left bottom)))
+	(label "VCC_3V3" (at 262.30 242.54 180) (fields_autoplaced yes)
+		(effects (font (size 1.27 1.27)) (justify left bottom)))
+	(label "GND" (at 275.00 252.70 270) (fields_autoplaced yes)
+		(effects (font (size 1.27 1.27)) (justify left bottom)))
+	(label "SD_MOSI" (at 287.70 242.54 0) (fields_autoplaced yes)
+		(effects (font (size 1.27 1.27)) (justify left bottom)))
+	(label "SD_SCK" (at 287.70 237.46 0) (fields_autoplaced yes)
+		(effects (font (size 1.27 1.27)) (justify left bottom)))
+	(label "VCC_3V3" (at 287.70 232.38 0) (fields_autoplaced yes)
+		(effects (font (size 1.27 1.27)) (justify left bottom)))
+	(label "VCC_3V3" (at 275.00 227.30 90) (fields_autoplaced yes)
+		(effects (font (size 1.27 1.27)) (justify left bottom)))
+	(label "VCC_3V3" (at 260.00 222.46 90) (fields_autoplaced yes)
+		(effects (font (size 1.27 1.27)) (justify left bottom)))
+	(label "GND" (at 260.00 227.54 270) (fields_autoplaced yes)
+		(effects (font (size 1.27 1.27)) (justify left bottom)))
+	(symbol (lib_id "Memory_Flash:W25Q128JV") (at 275.00 240.00 0) (unit 1)
+		(exclude_from_sim no) (in_bom yes) (on_board yes) (dnp no)
+		(property "Reference" "U12" (at 275.00 225.00 0) (effects (font (size 1.27 1.27))))
+		(property "Value" "W25Q128JVSIQ(Optional_Flash)" (at 275.00 255.00 0) (effects (font (size 1.27 1.27))))
+		(property "Footprint" "Package_SO:SOIC-8_208mil_WSON-8_8x6mm_DualCombo" (at 275.00 240.00 0) (hide yes) (effects (font (size 1.27 1.27))))
+		(property "Datasheet" "~" (at 275.00 240.00 0) (hide yes) (effects (font (size 1.27 1.27))))
+		(property "Description" "Dual-Footprint SPI NOR Flash 128Mb (Universal 4~128MB)" (at 275.00 240.00 0) (hide yes) (effects (font (size 1.27 1.27))))
+		(property "LCSC" "C97521" (at 275.00 240.00 0) (hide yes) (effects (font (size 1.27 1.27))))
+		(pin "1")
+		(pin "2")
+		(pin "3")
+		(pin "4")
+		(pin "5")
+		(pin "6")
+		(pin "7")
+		(pin "8")
+		(instances (project "epd_c6_slimbadge" (path "/00000000-0000-0000-0000-000000000001" (reference "U12") (unit 1))))
+	)
+	(symbol (lib_id "Device:C") (at 260.00 225.00 0) (unit 1)
+		(exclude_from_sim no) (in_bom yes) (on_board yes) (dnp no)
+		(property "Reference" "C35" (at 260.00 221.00 0) (effects (font (size 1.27 1.27))))
+		(property "Value" "0.1uF" (at 260.00 229.00 0) (effects (font (size 1.27 1.27))))
+		(property "Footprint" "Capacitor_SMD:C_0402_1005Metric" (at 260.00 225.00 0) (hide yes) (effects (font (size 1.27 1.27))))
+		(property "Datasheet" "~" (at 260.00 225.00 0) (hide yes) (effects (font (size 1.27 1.27))))
+		(property "Description" "Decoupling Capacitor for U12 Flash" (at 260.00 225.00 0) (hide yes) (effects (font (size 1.27 1.27))))
+		(property "LCSC" "C1525" (at 260.00 225.00 0) (hide yes) (effects (font (size 1.27 1.27))))
+		(pin "1")
+		(pin "2")
+		(instances (project "epd_c6_slimbadge" (path "/00000000-0000-0000-0000-000000000001" (reference "C35") (unit 1))))
+	)
 	(sheet_instances
