File: hardware/pcb_std/epd_c6_slimbadge.kicad_sch (KiCad schematic)
At the start: 90 parts, among them J1 Type-C_16P_MidMount, J2 SH1.0mm_2P_Battery, Q1 AO3400A, SW1 SK12D07, U1 ESP32-C6-MINI-1-N4, U10 ST25DV04K, U12 W25Q128JVSIQ(Optional_Flash), U2 USBLC6-2SC6, U3 CH224K, U4 SY6970, U5 ME6211C33M5G, U6 QMI8658C, U7 SHT40, U8 OPT3001, U9 PCF8563T, Y1 32.768kHz

Commit message: split
Parts:
- added J_NFC: FPC_0.5mm_4P, Connector_FFC-FPC:FPC_0.5mm_4P_Horizontal, symbol Connector_Generic:Conn_01x04
- ANT1_A, ANT1_B, J_EPD_A, J_EPD_B, PAD_BAT_N, PAD_BAT_P, TP1, TP2: now not fitted; now left out of the parts list
- C10, C11, C12, C13, C14, C6: LCSC C19702 -> C15849
- C18: LCSC C19702 -> C96446
- C19: LCSC C15850 -> C19702
- C2: LCSC C96123 -> C98192
- C3: LCSC C52923 -> C5137499
- C5: LCSC C22437 -> C15849
- D1, D3, D4: LCSC C22437 -> C77337
- J2: LCSC C160404 -> C41431902
- J_TF: value MicroSD_MidMount -> SIM-004X; LCSC C386341 -> C183629
- L1: LCSC C2993121 -> C497561
- L2: LCSC C408333 -> C98348
- LED1: LCSC C2890069 -> C2890035
- LED2: LCSC C84267 -> C51933292
- LED3: LCSC C84268 -> C84267
- LED4: LCSC C2286 -> C84265
- R10: LCSC C25905 -> C2906876
- R13: LCSC C25076 -> C2909315
- R22, R24, R5: LCSC C21190 -> C2906864
- SW1: value SK12D07 -> MSK-12C02; LCSC C432168 -> C431540
- U1: LCSC C5237255 -> C5736265
- U10: LCSC C444145 -> C2908287
- U12: value W25Q128JVSIQ(Optional_Flash) -> XT25F128; LCSC C97521 -> C42162960
- U3: LCSC C968262 -> C970725
- U4: LCSC C7438101 -> C5357542
- U5: LCSC C82942 -> C15651
- U6: LCSC C3038890 -> C3021082
- U7: value SHT40 -> AHT20; LCSC C271177 -> C2757850
- U8: LCSC C144888 -> C90462
- U9: value PCF8563T -> PCF8563DTR; LCSC C7787 -> C18723596
