File: hardware/pcb_lite/epd_c6_slimbadge.kicad_pcb (KiCad board)
At the start: 4 copper layers, 99 x 62 mm, 88 parts, among them J1 Type-C_16P, J2 JST_1.25mm_2P, Q1 AO3400A, SW1 SK12D07, U1 ESP32-C6-MINI-1, U10 ST25DV04K, U12 FLASH_4-128MB, U2 USBLC6-2SC6, U3 CH224K, U4 SY6970, U5 ME6211C33M5G, U6 QMI8658C, U7 SHT40, U8 OPT3001, U9 PCF8563T, Y1 32.768kHz

Commit message: v2.5
Parts:
- removed R10: 6.8k, Resistor_SMD:R_0402_1005Metric
- removed U3: CH224K, Package_SO:SSOP-10_3.9x4.9mm_P1.00mm
- added SW2: B3U-3000P, Button_Switch_SMD:SW_SPST_B3U-3000P, F.Cu at (13.5, 1.70)
- added TP1: VBUS, TestPoint:TestPoint_Pad_D1.2mm, F.Cu at (14.5, 7.00)
- added TP2: GND, TestPoint:TestPoint_Pad_D1.2mm, F.Cu at (17.5, 7.00)
- added TP3: 3V3, TestPoint:TestPoint_Pad_D1.2mm, F.Cu at (14.5, 9.50)
- added TP4: GND, TestPoint:TestPoint_Pad_D1.2mm, F.Cu at (17.5, 9.50)
- added TP5: BAT, TestPoint:TestPoint_Pad_D1.2mm, F.Cu at (14.5, 12.0)
- added TP6: BOOT, TestPoint:TestPoint_Pad_D1.2mm, F.Cu at (17.5, 12.0)
Routing:
- net GPIO9: track 0.00 -> 19.0 mm
- net VBUS: track 37.0 -> 54.5 mm
- net BAT_RAW: track 47.2 -> 55.2 mm
- net VCC_3V3: vias 30 -> 32
- net GND: vias 62 -> 66
